File: Yokai/Yokai-Choc/PCB/YokaiKeyboard.sch (KiCad schematic (older format))
At the start: 135 parts, among them J2 4PIN, J3 OLED, P1 i2c_pin, P2 i2c_pin, SW1 SW_PUSH-MX_W_LED, SW10 SW_PUSH-MX_W_LED, SW11 SW_PUSH-MX_W_LED, SW12 SW_PUSH-MX_W_LED, SW13 SW_PUSH-MX_W_LED, SW14 SW_PUSH-MX_W_LED, SW15 SW_PUSH-MX_W_LED, SW16 SW_PUSH-MX_W_LED, SW17 SW_PUSH-MX_W_LED, SW18 SW_PUSH-MX_W_LED, SW19 SW_PUSH-MX_W_LED, SW2 SW_PUSH-MX_W_LED, SW20 SW_PUSH-MX_W_LED, SW21 SW_PUSH-MX_W_LED, SW22 SW_PUSH-MX_W_LED, SW23 SW_PUSH-MX_W_LED, SW24 SW_PUSH-MX_W_LED, SW25 SW_PUSH-MX_W_LED, SW26 SW_PUSH-MX_W_LED, SW27 SW_PUSH-MX_W_LED, SW28 SW_PUSH-MX_W_LED, SW29 SW_PUSH-MX_W_LED, SW3 SW_PUSH-MX_W_LED, SW30 SW_PUSH-MX_W_LED, SW31 SW_PUSH-MX_W_LED, SW32 SW_PUSH-MX_W_LED, SW33 SW_PUSH-MX_W_LED, SW34 SW_PUSH-MX_W_LED, SW35 SW_PUSH-MX_W_LED, SW36 Rotary_Encoder, SW37 SW_PUSH-MX_W_LED, SW4 SW_PUSH-MX_W_LED, SW5 SW_PUSH-MX_W_LED, SW6 SW_PUSH-MX_W_LED, SW7 SW_PUSH-MX_W_LED, SW8 SW_PUSH-MX_W_LED, SW9 SW_PUSH-MX_W_LED, U1 nice_nano

Commit message: Add files via upload
*Increased pinky stagger
*Inverted stabilizer cutouts
*Added additional thumb key
*Minor footprint changes
Parts:
- added D37: D, Yokai:smd_diode, symbol Yokai:D-Yokai
- added L37: LED_sk2812_SM, Yokai:YS-SK6812MINI-E-DoubleSide, symbol Yokai:LED_sk2812_Mini_e
- added SW38: SW_PUSH-MX_W_LED, Yokai:Choc_Hotswap_DoubleSide, symbol keyboard_parts:SW_PUSH
- U1: symbol keebio:nice_nano -> Yokai:nice_nano
Connections:
- net GND: now also L37.3 (VSS)
- net VCC: now also L37.1 (VDD)
- net col1: now also SW38.1
- net row0: now also D1.1 (K), D2.1 (K), D3.1 (K), D4.1 (K), D5.1 (K), D6.1 (K)
- net row1: now also D10.1 (K), D11.1 (K), D12.1 (K), D13.1 (K), D8.1 (K), D9.1 (K)
- net row2: now also D15.1 (K), D16.1 (K), D17.1 (K), D18.1 (K), D19.1 (K), D20.1 (K)
- net row3: now also D22.1 (K), D23.1 (K), D24.1 (K), D25.1 (K), D26.1 (K), D27.1 (K)
- net row4: now also D29.1 (K), D30.1 (K), D31.1 (K), D32.1 (K), D33.1 (K), D34.1 (K)
- net row5: now also D37.1 (K)
- net at L30.4 (DIN): now also L37.2 (DOUT); no longer L23.2 (DOUT)
- new net: D37.2 (A), SW38.2
- new net: L23.2 (DOUT), L37.4 (DIN)
Other:
- moved on the sheet: D36
